File: pcb/minimum.kicad_pcb (KiCad board)
At the start: 2 copper layers, 16 x 20 mm, 26 parts, among them J1 USB4155-03-C_REVA, U1 RP2040, U2 SCD4x, U3 W25Q16JVUXIQ

Commit message: HIDING LABELS
Parts:
- moved C6 0.45 mm to (100.2, 65.0)
- moved C12 0.40 mm to (101.2, 65.0)
- moved C11 0.28 mm to (97.2, 65.0)
- moved R1 0.28 mm to (99.2, 65.0)
Changed lines of the file:
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@@
     (property "Sheetname" "")
     (attr smd)
-    (fp_text reference "C8" (at 0 -1.16) (layer "F.SilkS")
+    (fp_text reference "C8" (at 0 -1.16) (layer "F.SilkS") hide
       (effects (font (size 1 1) (thickness 0.15)))
     )
@@
     (property "Sheetname" "")
     (attr smd)
-    (fp_text reference "R6" (at 0 -1.17) (layer "F.SilkS")
+    (fp_text reference "R6" (at 0 -1.17) (layer "F.SilkS") hide
       (effects (font (size 1 1) (thickness 0.15)))
     )
@@
     (property "Sheetname" "")
     (attr smd)
-    (fp_text reference "C16" (at 0 -1.16) (layer "F.SilkS")
+    (fp_text reference "C16" (at 0 -1.16) (layer "F.SilkS") hide
       (effects (font (size 1 1) (thickness 0.15)))
     )
@@
     (property "Sheetname" "")
     (attr smd)
-    (fp_text reference "C9" (at 0 -1.16) (layer "F.SilkS")
+    (fp_text reference "C9" (at 0 -1.16) (layer "F.SilkS") hide
       (effects (font (size 1 1) (thickness 0.15)))
     )
@@
     (property "Sheetname" "")
     (attr smd)
-    (fp_text reference "C15" (at 0 1.16) (layer "B.SilkS")
+    (fp_text reference "C15" (at 0 1.16) (layer "B.SilkS") hide
       (effects (font (size 1 1) (thickness 0.15)) (justify mirror))
     )
@@
     (property "Sheetname" "")
     (attr smd)
-    (fp_text reference "C7" (at 0 1.16) (layer "B.SilkS")
+    (fp_text reference "C7" (at 0 1.16) (layer "B.SilkS") hide
       (effects (font (size 1 1) (thickness 0.15)) (justify mirror))
     )
@@
     (property "Sheetname" "")
     (attr smd)
-    (fp_text reference "C10" (at 0 1.16) (layer "B.SilkS")
+    (fp_text reference "C10" (at 0 1.16) (layer "B.SilkS") hide
       (effects (font (size 1 1) (thickness 0.15)) (justify mirror))
     )
@@
     (property "Sheetname" "")
     (attr smd)
-    (fp_text reference "R4" (at 0 1.17 90) (layer "B.SilkS")
+    (fp_text reference "R4" (at 0 1.17 90) (layer "B.SilkS") hide
       (effects (font (size 1 1) (thickness 0.15)) (justify mirror))
     )
@@
   )
   (footprint "Capacitor_SMD:C_0402_1005Metric" (layer "B.Cu")
-    (at 97 64.8 90)
+    (at 97.2 65 90)
     (descr "Capacitor SMD 0402 (1005 Metric), square (rectangular) end terminal, IPC_7351 nominal, (Body size source: IPC-SM-782 page 76, https://www.pcb-3d.com/wordpress/wp-content/uploads/ipc-sm-782a_amendment_1_and_2.pdf), generated with kicad-footprint-generator")
     (tags "capacitor")
@@
     (property "Sheetname" "")
     (attr smd)
-    (fp_text reference "C11" (at 0 1.16 90) (layer "B.SilkS")
+    (fp_text reference "C11" (at 0 1.16 90) (layer "B.SilkS") hide
       (effects (font (size 1 1) (thickness 0.15)) (justify mirror))
     )
@@
   )
   (footprint "Resistor_SMD:R_0402_1005Metric" (layer "B.Cu")
-    (at 99 64.8 -90)
+    (at 99.2 65 -90)
     (descr "Resistor SMD 0402 (1005 Metric), square (rectangular) end terminal, IPC_7351 nominal, (Body size source: IPC-SM-782 page 72, https://www.pcb-3d.com/wordpress/wp-content/uploads/ipc-sm-782a_amendment_1_and_2.pdf), generated with kicad-footprint-generator")
     (tags "resistor")
@@
     (property "Sheetname" "")
     (attr smd)
-    (fp_text reference "R1" (at 0 1.17 90) (layer "B.SilkS")
+    (fp_text reference "R1" (at 0 1.17 90) (layer "B.SilkS") hide
       (effects (font (size 1 1) (thickness 0.15)) (justify mirror))
     )
@@
     (property "Sheetname" "")
     (attr smd)
-    (fp_text reference "C14" (at 0 1.16) (layer "B.SilkS")
+    (fp_text reference "C14" (at 0 1.16) (layer "B.SilkS") hide
       (effects (font (size 1 1) (thickness 0.15)) (justify mirror))
     )
@@
     (property "Sheetname" "")
     (attr smd)
-    (fp_text reference "C1" (at 0 1.16) (layer "B.SilkS")
+    (fp_text reference "C1" (at 0 1.16) (layer "B.SilkS") hide
       (effects (font (size 1 1) (thickness 0.15)) (justify mirror))
     )
@@
     (property "Sheetname" "")
     (attr smd)
-    (fp_text reference "R5" (at 0 1.17 90) (layer "B.SilkS")
+    (fp_text reference "R5" (at 0 1.17 90) (layer "B.SilkS") hide
       (effects (font (size 1 1) (thickness 0.15)) (justify mirror))
     )
@@
     (property "Sheetfile" "minimum.kicad_sch")
     (property "Sheetname" "")
-    (fp_text reference "U3" (at 0 0) (layer "B.SilkS")
-      (effects (font (size 1 1) (thickness 0.15)) (justify mirror))
-    )
-    (fp_text value "W25Q16JVUXIQ" (at 0 0) (layer "B.SilkS")
+    (fp_text reference "U3" (at 0 -0.6) (layer "B.SilkS")
+      (effects (font (size 0.6 0.6) (thickness 0.15)) (justify mirror))
+    )
+    (fp_text value "W25Q16JVUXIQ" (at 0 0) (layer "B.SilkS") hide
       (effects (font (size 1 1) (thickness 0.15)) (justify mirror))
     )
@@
     (fp_circle (center -0.992 0.75) (end -0.9158 0.75) (layer "B.Fab") (width 0.1) (fill none))
     (pad "1" smd rect locked (at -1.3984 0.750001 180) (size 0.8128 0.254) (layers "B.Cu" "B.Paste" "B.Mask")
-      (net 18 "/QSPI_SS") (pinfunction "CS") (pintype "input"))
+      (net 18 "/QSPI_SS") (pinfunction "CS"))
     (pad "2" smd rect locked (at -1.3984 0.25 180) (size 0.8128 0.254) (layers "B.Cu" "B.Paste" "B.Mask")
-      (net 17 "/QSPI_SD1") (pinfunction "DO_IO1") (pintype "bidirectional"))
+      (net 17 "/QSPI_SD1") (pinfunction "DO_IO1"))
     (pad "3" smd rect locked (at -1.3984 -0.25 180) (size 0.8128 0.254) (layers "B.Cu" "B.Paste" "B.Mask")
-      (net 16 "/QSPI_SD2") (pinfunction "IO2") (pintype "bidirectional"))
+      (net 16 "/QSPI_SD2") (pinfunction "IO2"))
     (pad "4" smd rect locked (at -1.3984 -0.750001 180) (size 0.8128 0.254) (layers "B.Cu" "B.Paste" "B.Mask")
-      (net 3 "GND") (pinfunction "GND") (pintype "power_in"))
+      (net 3 "GND") (pinfunction "GND"))
     (pad "5" smd rect locked (at 1.3984 -0.750001 180) (size 0.8128 0.254) (layers "B.Cu" "B.Paste" "B.Mask")
-      (net 15 "/QSPI_SD0") (pinfunction "DI_IO0") (pintype "bidirectional"))
+      (net 15 "/QSPI_SD0") (pinfunction "DI_IO0"))
     (pad "6" smd rect locked (at 1.3984 -0.25 180) (size 0.8128 0.254) (layers "B.Cu" "B.Paste" "B.Mask")
-      (net 14 "/QSPI_SCLK") (pinfunction "CLK") (pintype "input"))
+      (net 14 "/QSPI_SCLK") (pinfunction "CLK"))
     (pad "7" smd rect locked (at 1.3984 0.25 180) (size 0.8128 0.254) (layers "B.Cu" "B.Paste" "B.Mask")
-      (net 13 "/QSPI_SD3") (pinfunction "IO3") (pintype "bidirectional"))
+      (net 13 "/QSPI_SD3") (pinfunction "IO3"))
     (pad "8" smd rect locked (at 1.3984 0.750001 180) (size 0.8128 0.254) (layers "B.Cu" "B.Paste" "B.Mask")
-      (net 2 "+3V3") (pinfunction "VCC") (pintype "power_in"))
+      (net 2 "+3V3") (pinfunction "VCC"))
     (pad "9" smd rect (at 0 0 180) (size 0.2032 1.6002) (layers "B.Cu" "B.Paste" "B.Mask"))
     (model "${KIPRJMOD}/3Dshapes/W25Q16JVUXIQ_WIN.step"
@@
     (property "Sheetname" "")
     (attr smd)
-    (fp_text reference "R3" (at 0 1.17) (layer "B.SilkS")
+    (fp_text reference "R3" (at 0 1.17) (layer "B.SilkS") hide
       (effects (font (size 1 1) (thickness 0.15)) (justify mirror))
     )
@@
   )
   (footprint "Capacitor_SMD:C_0402_1005Metric" (layer "B.Cu")
-    (at 101.2 64.6 90)
+    (at 101.2 65 90)
     (descr "Capacitor SMD 0402 (1005 Metric), square (rectangular) end terminal, IPC_7351 nominal, (Body size source: IPC-SM-782 page 76, https://www.pcb-3d.com/wordpress/wp-content/uploads/ipc-sm-782a_amendment_1_and_2.pdf), generated with kicad-footprint-generator")
     (tags "capacitor")
@@
     (property "Sheetname" "")
     (attr smd)
-    (fp_text reference "C12" (at 0 1.16 90) (layer "B.SilkS")
+    (fp_text reference "C12" (at 0 1.16 90) (layer "B.SilkS") hide
       (effects (font (size 1 1) (thickness 0.15)) (justify mirror))
     )
@@
     (property "Sheetname" "")
     (attr smd)
-    (fp_text reference "C2" (at 0 1.16) (layer "B.SilkS")
+    (fp_text reference "C2" (at 0 1.16) (layer "B.SilkS") hide
       (effects (font (size 1 1) (thickness 0.15)) (justify mirror))
     )
@@
     (attr smd)
     (fp_text reference "U1" (at 0 4.82) (layer "B.SilkS")
-      (effects (font (size 1 1) (thickness 0.15)) (justify mirror))
+      (effects (font (size 0.6 0.6) (thickness 0.15)) (justify mirror))
     )
     (fp_text value "RP2040" (at 0 -4.82) (layer "B.Fab")
@@
     (property "Sheetname" "")
     (attr smd)
-    (fp_text reference "C4" (at 0 1.16) (layer "B.SilkS")
+    (fp_text reference "C4" (at 0 1.16) (layer "B.SilkS") hide
       (effects (font (size 1 1) (thickness 0.15)) (justify mirror))
     )
@@
     (property "Sheetname" "")
     (attr smd)
-    (fp_text reference "R2" (at 0 1.17 90) (layer "B.SilkS")
+    (fp_text reference "R2" (at 0 1.17 90) (layer "B.SilkS") hide
       (effects (font (size 1 1) (thickness 0.15)) (justify mirror))
     )
@@
     (property "Sheetname" "")
     (attr smd)
-    (fp_text reference "C13" (at 0 1.16) (layer "B.SilkS")
+    (fp_text reference "C13" (at 0 1.16) (layer "B.SilkS") hide
       (effects (font (size 1 1) (thickness 0.15)) (justify mirror))
     )
@@
   )
   (footprint "Capacitor_SMD:C_0402_1005Metric" (layer "B.Cu")
-    (at 100 64.6 90)
+    (at 100.2 65 90)
     (descr "Capacitor SMD 0402 (1005 Metric), square (rectangular) end terminal, IPC_7351 nominal, (Body size source: IPC-SM-782 page 76, https://www.pcb-3d.com/wordpress/wp-content/uploads/ipc-sm-782a_amendment_1_and_2.pdf), generated with kicad-footprint-generator")
     (tags "capacitor")
@@
     (property "Sheetname" "")
     (attr smd)
-    (fp_text reference "C6" (at 0 1.16 90) (layer "B.SilkS")
+    (fp_text reference "C6" (at 0 1.16 90) (layer "B.SilkS") hide
       (effects (font (size 1 1) (thickness 0.15)) (justify mirror))
     )
@@
     (property "Sheetname" "")
     (attr smd)
-    (fp_text reference "C5" (at 0 1.16) (layer "B.SilkS")
-      (effects (font (size 1 1) (thickness 0.15)) (justify mirror))
-    )
+    (fp_text reference "C5" (at 0 1.16) (layer "B.SilkS") hide
+      (effects (font (size 1 1) (thickness 0.15)) (justify mirror))
+    )

Commit message: routing
Parts:
- added C17: 10u, Capacitor_SMD:C_0603_1608Metric, F.Cu at (106.4, 62.0)
- added C18: 10u, Capacitor_SMD:C_0603_1608Metric, F.Cu at (93.4, 68.4)
- added R7: 10k, Resistor_SMD:R_0402_1005Metric, F.Cu at (96.0, 65.5)
- added U4: XCL220, SMD:XCL220, F.Cu at (94.0, 65.4)
- added Y1: C2E-12.000-18-1020-X-R, SMD:AKER_C2E, B.Cu at (101.2, 77.2)
- R3, R4: moved to F.Cu
- moved C5 4.34 mm to (97.2, 77.4)
- moved R3 3.31 mm to (100.6, 78.8), turned to 0 degrees
- moved C9 2.81 mm to (98.0, 78.8)
- moved C15 2.63 mm to (98.6, 78.4)
- moved C14 1.92 mm to (103.4, 76.9), turned to -90 degrees
- moved C16 1.80 mm to (105.2, 64.6)
- moved R4 1.68 mm to (103.2, 78.8), turned to 180 degrees
- moved U2 1.30 mm to (100.0, 72.6)
- moved C8 1.23 mm to (97.7, 65.5), turned to 90 degrees
- moved R5 0.68 mm to (99.0, 76.9)
- moved C13 0.63 mm to (97.2, 76.4)
- moved C1 0.28 mm to (94.6, 68.6)
- moved C2 0.20 mm to (94.6, 72.4)
Connections:
- net Net-(R3-Pad2) renamed /SCL
- net Net-(R4-Pad2) renamed /SDA
- J1 pad A4: Net-(J1-PadA4) -> VBUS
- J1 pad A9: Net-(J1-PadA4) -> VBUS
- J1 pad B4: Net-(J1-PadB4) -> VBUS
- J1 pad B9: Net-(J1-PadB4) -> VBUS
Routing:
- net +3V3: track 0.00 -> 39.6 mm, vias 0 -> 10
- net GND: track 0.00 -> 20.7 mm, vias 0 -> 10
- net +1V1: track 0.00 -> 19.0 mm
- net /QSPI_SS: track 0.00 -> 9.38 mm, vias 0 -> 1
- net /QSPI_SD1: track 0.00 -> 7.81 mm
- net /XIN: track 0.00 -> 5.69 mm
- net /QSPI_SD2: track 0.00 -> 5.65 mm
- net /QSPI_SD3: track 0.00 -> 4.30 mm
- net /QSPI_SCLK: track 0.00 -> 3.63 mm
- net /QSPI_SD0: track 0.00 -> 2.96 mm
- net /XOUTc: track 0.00 -> 2.82 mm
- net /XOUT: track 0.00 -> 2.34 mm
- net /SDA: track 0.00 -> 1.93 mm
- net /SCL: track 0.00 -> 1.92 mm
- net Net-(U4-Pad1): track 0.00 -> 1.51 mm
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- added copper zone on In1.Cu, net +3V3
- added copper zone on B.Cu, net GND
- added copper zone on F.Cu, net GND
- added copper zone on In2.Cu, net GND
Other:
- copper layers 2 -> 4

Commit message: routing
Parts:
- moved R3 6.67 mm to (106.5, 75.6), turned to -90 degrees
- moved C9 5.37 mm to (93.5, 75.8), turned to 90 degrees
- moved R4 3.48 mm to (106.5, 77.6), turned to 90 degrees
- moved C10 0.70 mm to (94.5, 66.0)
- moved C7 0.70 mm to (94.5, 67.0)
Connections:
- U1 pad 13: (no net) -> /SDA
- U1 pad 14: (no net) -> /SCL
Routing:
- net /SDA: track 1.93 -> 7.99 mm, vias 0 -> 1
- net /SCL: track 1.92 -> 7.77 mm, vias 0 -> 1
- net VBUS: track 0.00 -> 3.21 mm
- net +3V3: track 39.6 -> 42.3 mm, vias 10 -> 11
- net GND: track 20.7 -> 18.6 mm, vias 10 -> 11
- net Net-(U4-Pad1): track 1.51 -> 0.79 mm

Commit message: routing
Parts:
- U3: value W25Q16JVUXIQ -> W25Q16JVUXIQ_WIN
- moved C6 0.13 mm to (100.3, 64.9)
- moved R2 0.12 mm to (98.3, 65.0)
- moved C12 0.12 mm to (101.3, 64.9)
- moved C11 0.10 mm to (97.3, 65.0)
- moved R1 0.09 mm to (99.3, 65.0)
Connections:
- net Net-(R1-Pad2) renamed /Pi_USB_D+
- net Net-(R2-Pad1) renamed /Pi_USB_D-
Routing:
- net /Pi_USB_D-: track 0.00 -> 2.42 mm
- net /Pi_USB_D+: track 0.00 -> 2.42 mm
- net VBUS: track 3.21 -> 1.60 mm
- net +1V1: track 18.9 -> 19.8 mm
- net GND: track 18.6 -> 19.4 mm, vias 11 -> 12
- net +3V3: track 42.3 -> 42.4 mm, vias 11 -> 12
